File: Nixie Board.sch (EAGLE design)
At the start: 39 parts, among them Q1 DXTA92-13, Q10 SXTA42TA, Q2 SXTA42TA, Q3 DXTA92-13, Q4 SXTA42TA, Q5 DXTA92-13, Q6 SXTA42TA, Q7 DXTA92-13, Q8 SXTA42TA, Q9 DXTA92-13

Commit message: chore: added bom and MPN to components
Parts:
- J1, J2: MPN (none) -> INS-1
- JP1: MPN (none) -> 30314-6002HB
- NX1, NX2, NX3, NX4: MPN (none) -> IN-12B
- R1, R11, R12, R13, R15, R16, R17, R19, R20, R3, R4, R5, R7, R8, R9: MPN (none) -> ESR03EZPJ103
- R10, R14, R18, R2, R6: MPN (none) -> ERJ-3EKF1004V
- U$1: MPN (none) -> K155ID1
- U$2: MPN (none) -> NCH8200HV
Other:
- note added: "K155ID1"
- note added: "NCH8200HV"
- note added: "Used ISDCB84 Ribbon Cable"
